File: Master_PSoC5LP/eagle/RhythmMachine-Master/RhythmMachine-Master.brd (EAGLE design)
At the start: 94.9 x 72.4 mm, 29 parts, among them SW1 EC12E_SW, SW2 EC12E_SW, SW3 EC12E_SW

Commit message: Master_PSoC5LP: Eagleファイル: 基板図を作成
Parts:
- removed U$4: AK_TCTSW, mylib:TME1
- added TP4: TPPAD1-13, testpad:P1-13
- moved TP1 62.3 mm to (66.0, 20.3)
- moved TP2 11.4 mm to (63.5, 20.3)
- moved JP3 10.2 mm to (55.9, -1.27)
- moved JP2 7.62 mm to (64.8, -1.27)
- moved R4 7.62 mm to (34.3, 10.2), turned to 180 degrees
- moved TP3 5.08 mm to (2.54, 48.3)
- moved U$2 5.08 mm to (83.8, 49.5), turned to 180 degrees
- moved U$3 5.08 mm to (83.8, 59.7), turned to 180 degrees
Connections:
- removed net SCL: JP1.4, U$1.50
- removed net SDA: JP1.5, U$1.49
- new net I2C_SCL: JP1.4, U$1.49
- new net I2C_SDA: JP1.5, U$1.50
- net GND: now also U$2.1; no longer U$2.6, U$4.6
- net LED_B: now also U$1.36; no longer U$1.35
- net LED_G: now also U$1.37; no longer U$1.36
- net LED_R: now also U$1.35; no longer U$1.37
- net N$6: now also RCA_HOT.2; no longer RCA_HOT.1
- net SW1: now also U$2.3; no longer U$2.4
- net SW3: no longer U$4.4
- net VDAC8_2: now also TP4.TP
Routing:
- net GND: track 0.00 -> 332.9 mm
- net VCCIO: track 0.00 -> 197.5 mm
- net CONTR: track 0.00 -> 94.2 mm
- net LED_R: track 0.00 -> 76.2 mm
- net LED_B: track 0.00 -> 63.5 mm
- net LED_G: track 0.00 -> 55.9 mm
- net I2C_RST: track 0.00 -> 50.8 mm
- net I2C_SCL: track 0.00 -> 45.7 mm
- net I2C_SDA: track 0.00 -> 40.6 mm
- net RE1_A: track 0.00 -> 39.0 mm
- net RE1_B: track 0.00 -> 35.0 mm
- net SS2: track 0.00 -> 30.6 mm
- net SS1: track 0.00 -> 30.6 mm
- net SCK: track 0.00 -> 30.6 mm
- net MOSI: track 0.00 -> 30.6 mm
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
Commit message: Eagle: 修正
Parts:
- R1, R2: value (none) -> 1k
- R3: value (none) -> 1.5k
- R4, R6: value (none) -> 220
- R5: value (none) -> 10k
- moved TP4 14.8 mm to (20.3, 55.9)
Connections:
- net VDAC8_1: now also U$1.22; no longer R6.2, U$1.23
- net VDAC8_2: now also R6.2, U$1.23; no longer U$1.24
Routing:
- net VDAC8_2: track 2.54 -> 40.2 mm
- net VDAC8_1: track 30.5 -> 15.2 mm
- net CONTR: track 94.2 -> 88.7 mm
- net LED_R: track 76.2 -> 81.3 mm
- net LED_B: track 63.5 -> 68.6 mm
- net LED_G: track 55.9 -> 58.4 mm
- net SS1: track 30.6 -> 31.3 mm
- net SCK: track 30.6 -> 31.3 mm
- net MOSI: track 30.6 -> 31.3 mm
- net MISO: track 30.6 -> 31.3 mm
- net SS2: track 30.6 -> 31.3 mm

Commit message: Eagleファイル修正
Connections:
- removed net SW3: U$1.4
- removed net SW4: U$1.5
Routing:
- net VCCIO: track 197.5 -> 164.5 mm
Changed lines of the file:
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@@
 <wire x1="68.58" y1="55.88" x2="81.28" y2="55.88" width="0.4064" layer="16"/>
-</signal>
-<signal name="SW3">
-<contactref element="U$1" pad="4"/>
-</signal>
-<signal name="SW4">
-<contactref element="U$1" pad="5"/>
 </signal>
 <signal name="VCCIO">
@@
 <contactref element="TP1" pad="TP"/>
 <wire x1="91.44" y1="43.18" x2="93.98" y2="43.18" width="0.4064" layer="16"/>
-<wire x1="93.98" y1="30.48" x2="66.04" y2="30.48" width="0.4064" layer="16"/>
-<wire x1="66.04" y1="30.48" x2="66.04" y2="25.4" width="0.4064" layer="16"/>
 <wire x1="83.82" y1="7.62" x2="93.98" y2="17.78" width="0.4064" layer="16"/>
-<wire x1="93.98" y1="17.78" x2="93.98" y2="30.48" width="0.4064" layer="16"/>
-<wire x1="93.98" y1="30.48" x2="93.98" y2="43.18" width="0.4064" layer="16"/>
+<wire x1="93.98" y1="17.78" x2="93.98" y2="43.18" width="0.4064" layer="16"/>
 <wire x1="66.04" y1="25.4" x2="66.04" y2="20.32" width="0.4064" layer="16"/>
 <wire x1="66.04" y1="20.32" x2="66.04" y2="2.54" width="0.4064" layer="16"/>
