File: Master_PSoC5LP/eagle/RhythmMachine-Master/RhythmMachine-Master.sch (EAGLE design)
At the start: 29 parts, among them SW1 EC12E_SW, SW2 EC12E_SW, SW3 EC12E_SW

Commit message: Master_PSoC5LP: Eagleファイル: 基板図を作成
Parts:
- removed U$4: AK_TCTSW, mylib:AK_TCTSW
- added TP4: TPPAD1-13, testpad:TPPAD1-13
Connections:
- removed net SCL: JP1.4, U$1.50
- removed net SDA: JP1.5, U$1.49
- new net I2C_SCL: JP1.4, U$1.49
- new net I2C_SDA: JP1.5, U$1.50
- net GND: now also U$2.P; no longer U$2.P@1, U$4.P@1
- net LED_B: now also U$1.36; no longer U$1.35
- net LED_G: now also U$1.37; no longer U$1.36
- net LED_R: now also U$1.35; no longer U$1.37
- net N$6: now also RCA_HOT.2; no longer RCA_HOT.1
- net SW1: now also U$2.S; no longer U$2.S@1
- net SW3: no longer U$4.S@1
- net VDAC8_2: now also TP4.TP
Other:
- moved on the sheet: RCA_GND, RCA_HOT, TP3
Changed lines of the file:
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@@
 <part name="SUPPLY21" library="supply2" deviceset="GND" device=""/>
 <part name="C1" library="rcl" deviceset="CPOL-EU" device="E2.5-7"/>
-<part name="U$4" library="mylib" deviceset="AK_TCTSW" device=""/>
-<part name="SUPPLY11" library="supply2" deviceset="GND" device=""/>
 <part name="RCA_HOT" library="pinhead" deviceset="PINHD-1X6" device=""/>
 <part name="RCA_GND" library="pinhead" deviceset="PINHD-1X6" device=""/>
@@
 <part name="TP2" library="testpad" deviceset="TP" device="PAD1-13"/>
 <part name="TP3" library="testpad" deviceset="TP" device="PAD1-13"/>
+<part name="TP4" library="testpad" deviceset="TP" device="PAD1-13"/>
 </parts>
 <sheets>
@@
 <instance part="SUPPLY3" gate="GND" x="33.02" y="93.98"/>
 <instance part="SUPPLY4" gate="GND" x="43.18" y="30.48"/>
-<instance part="SUPPLY5" gate="G$1" x="33.02" y="48.26"/>
+<instance part="SUPPLY5" gate="G$1" x="30.48" y="48.26"/>
 <instance part="VCC1" gate="G$1" x="88.9" y="106.68"/>
 <instance part="FRAME1" gate="G$1" x="0" y="0"/>
@@
 <instance part="U$2" gate="G$1" x="119.38" y="114.3"/>
 <instance part="U$3" gate="G$1" x="137.16" y="114.3"/>
-<instance part="SUPPLY9" gate="GND" x="121.92" y="106.68"/>
+<instance part="SUPPLY9" gate="GND" x="119.38" y="106.68"/>
 <instance part="SUPPLY10" gate="GND" x="139.7" y="106.68"/>
 <instance part="RGB_LED" gate="A" x="142.24" y="78.74"/>
@@
 <instance part="SUPPLY21" gate="GND" x="160.02" y="33.02"/>
 <instance part="C1" gate="G$1" x="167.64" y="55.88" rot="R90"/>
-<instance part="U$4" gate="G$1" x="154.94" y="114.3"/>
-<instance part="SUPPLY11" gate="GND" x="157.48" y="106.68"/>
-<instance part="RCA_HOT" gate="A" x="180.34" y="48.26"/>
-<instance part="RCA_GND" gate="A" x="205.74" y="48.26"/>
+<instance part="RCA_HOT" gate="A" x="180.34" y="50.8"/>
+<instance part="RCA_GND" gate="A" x="205.74" y="50.8"/>
 <instance part="H1" gate="G$1" x="88.9" y="22.86"/>
 <instance part="H2" gate="G$1" x="88.9" y="15.24"/>
@@
 <instance part="TP1" gate="G$1" x="93.98" y="106.68"/>
 <instance part="TP2" gate="G$1" x="93.98" y="93.98" rot="R180"/>
-<instance part="TP3" gate="G$1" x="27.94" y="50.8"/>
+<instance part="TP3" gate="G$1" x="25.4" y="50.8"/>
+<instance part="TP4" gate="G$1" x="35.56" y="50.8"/>
 </instances>
 <busses>
@@
 </segment>
 <segment>
-<pinref part="U$2" gate="G$1" pin="P@1"/>
-<pinref part="SUPPLY9" gate="GND" pin="GND"/>
-</segment>
-<segment>
 <pinref part="U$3" gate="G$1" pin="P@1"/>
 <pinref part="SUPPLY10" gate="GND" pin="GND"/>
@@
 <segment>
 <pinref part="SUPPLY20" gate="GND" pin="GND"/>
-<wire x1="190.5" y1="35.56" x2="190.5" y2="43.18" width="0.1524" layer="91"/>
+<wire x1="190.5" y1="35.56" x2="190.5" y2="45.72" width="0.1524" layer="91"/>
 <pinref part="RCA_GND" gate="A" pin="6"/>
-<wire x1="203.2" y1="43.18" x2="190.5" y2="43.18" width="0.1524" layer="91"/>
+<wire x1="203.2" y1="45.72" x2="190.5" y2="45.72" width="0.1524" layer="91"/>
 </segment>
 <segment>
 <pinref part="LED1" gate="G$1" pin="C"/>
 <pinref part="SUPPLY21" gate="GND" pin="GND"/>
-</segment>
-<segment>
-<pinref part="U$4" gate="G$1" pin="P@1"/>
-<pinref part="SUPPLY11" gate="GND" pin="GND"/>
 </segment>
 <segment>
@@
 <wire x1="30.48" y1="111.76" x2="30.48" y2="114.3" width="0.1524" layer="91"/>
 </segment>
+<segment>
+<pinref part="U$2" gate="G$1" pin="P"/>
+<pinref part="SUPPLY9" gate="GND" pin="GND"/>
+</segment>
 </net>
 <net name="VDD" class="0">
 <segment>
 <pinref part="SUPPLY5" gate="G$1" pin="VDD"/>
-<wire x1="33.02" y1="45.72" x2="33.02" y2="38.1" width="0.1524" layer="91"/>
+<wire x1="30.48" y1="45.72" x2="30.48" y2="38.1" width="0.1524" layer="91"/>
 <pinref part="U$1" gate="G$1" pin="26"/>
-<wire x1="33.02" y1="38.1" x2="50.8" y2="38.1" width="0.1524" layer="91"/>
+<wire x1="30.48" y1="38.1" x2="50.8" y2="38.1" width="0.1524" layer="91"/>
 <pinref part="TP3" gate="G$1" pin="TP"/>
-<wire x1="27.94" y1="48.26" x2="27.94" y2="38.1" width="0.1524" layer="91"/>
-<wire x1="33.02" y1="38.1" x2="27.94" y2="38.1" width="0.1524" layer="91"/>
-<junction x="33.02" y="38.1"/>
-</segment>
-</net>
-<net name="SCL" class="0">
-<segment>
-<pinref part="U$1" gate="G$1" pin="50"/>
-<wire x1="66.04" y1="96.52" x2="81.28" y2="96.52" width="0.1524" layer="91"/>
-<label x="68.58" y="96.52" size="1.778" layer="95"/>
-</segment>
-<segment>
-<pinref part="JP1" gate="A" pin="4"/>
-<wire x1="220.98" y1="127" x2="205.74" y2="127" width="0.1524" layer="91"/>
-<label x="205.74" y="127" size="1.778" layer="95"/>
-</segment>
-</net>
-<net name="SDA" class="0">
-<segment>
-<pinref part="U$1" gate="G$1" pin="49"/>
-<wire x1="66.04" y1="93.98" x2="81.28" y2="93.98" width="0.1524" layer="91"/>
-<label x="68.58" y="93.98" size="1.778" layer="95"/>
-</segment>
-<segment>
-<pinref part="JP1" gate="A" pin="5"/>
-<wire x1="220.98" y1="124.46" x2="205.74" y2="124.46" width="0.1524" layer="91"/>
-<label x="205.74" y="124.46" size="1.778" layer="95"/>
+<wire x1="25.4" y1="48.26" x2="25.4" y2="38.1" width="0.1524" layer="91"/>
+<wire x1="30.48" y1="38.1" x2="25.4" y2="38.1" width="0.1524" layer="91"/>
+<junction x="30.48" y="38.1"/>
 </segment>
 </net>
@@
 <segment>
 <pinref part="U$1" gate="G$1" pin="24"/>
-<wire x1="50.8" y1="43.18" x2="38.1" y2="43.18" width="0.1524" layer="91"/>
+<wire x1="50.8" y1="43.18" x2="35.56" y2="43.18" width="0.1524" layer="91"/>
 <label x="38.1" y="43.18" size="1.778" layer="95"/>
+<pinref part="TP4" gate="G$1" pin="TP"/>
+<wire x1="35.56" y1="48.26" x2="35.56" y2="43.18" width="0.1524" layer="91"/>
 </segment>
 </net>
@@
 </segment>
 <segment>
-<pinref part="U$2" gate="G$1" pin="S@1"/>
-<wire x1="121.92" y1="119.38" x2="121.92" y2="124.46" width="0.1524" layer="91"/>
-<label x="121.92" y="121.92" size="1.778" layer="95" rot="R90"/>
+<pinref part="U$2" gate="G$1" pin="S"/>
+<wire x1="119.38" y1="119.38" x2="119.38" y2="124.46" width="0.1524" layer="91"/>
+<label x="119.38" y="121.92" size="1.778" layer="95" rot="R90"/>
 </segment>
 </net>
@@
 <wire x1="38.1" y1="93.98" x2="50.8" y2="93.98" width="0.1524" layer="91"/>
 <label x="38.1" y="93.98" size="1.778" layer="95"/>
-</segment>
-<segment>
-<pinref part="U$4" gate="G$1" pin="S@1"/>
-<wire x1="157.48" y1="119.38" x2="157.48" y2="124.46" width="0.1524" layer="91"/>
-<label x="157.48" y="121.92" size="1.778" layer="95" rot="R90"/>
 </segment>
 </net>
@@
 <net name="LED_R" class="0">
 <segment>
+<pinref part="R3" gate="G$1" pin="1"/>
+<wire x1="124.46" y1="76.2" x2="109.22" y2="76.2" width="0.1524" layer="91"/>
+<label x="109.22" y="76.2" size="1.778" layer="95"/>
+</segment>
+<segment>
+<pinref part="U$1" gate="G$1" pin="35"/>
+<wire x1="66.04" y1="58.42" x2="81.28" y2="58.42" width="0.1524" layer="91"/>
+<label x="68.58" y="58.42" size="1.778" layer="95"/>
+</segment>
+</net>
+<net name="LED_G" class="0">
+<segment>
+<pinref part="R1" gate="G$1" pin="1"/>
+<wire x1="124.46" y1="83.82" x2="109.22" y2="83.82" width="0.1524" layer="91"/>
+<label x="109.22" y="83.82" size="1.778" layer="95"/>
+</segment>
+<segment>
 <pinref part="U$1" gate="G$1" pin="37"/>
 <wire x1="66.04" y1="63.5" x2="81.28" y2="63.5" width="0.1524" layer="91"/>
 <label x="68.58" y="63.5" size="1.778" layer="95"/>
 </segment>
-<segment>
-<pinref part="R3" gate="G$1" pin="1"/>
-<wire x1="124.46" y1="76.2" x2="109.22" y2="76.2" width="0.1524" layer="91"/>
-<label x="109.22" y="76.2" size="1.778" layer="95"/>
-</segment>
-</net>
-<net name="LED_G" class="0">
+</net>
+<net name="LED_B" class="0">
+<segment>
+<pinref part="R2" gate="G$1" pin="1"/>
+<wire x1="116.84" y1="81.28" x2="109.22" y2="81.28" width="0.1524" layer="91"/>
+<label x="109.22" y="81.28" size="1.778" layer="95"/>
+</segment>
 <segment>
 <pinref part="U$1" gate="G$1" pin="36"/>
 <wire x1="66.04" y1="60.96" x2="81.28" y2="60.96" width="0.1524" layer="91"/>
 <label x="68.58" y="60.96" size="1.778" layer="95"/>
-</segment>
-<segment>
-<pinref part="R1" gate="G$1" pin="1"/>
-<wire x1="124.46" y1="83.82" x2="109.22" y2="83.82" width="0.1524" layer="91"/>
-<label x="109.22" y="83.82" size="1.778" layer="95"/>
-</segment>
-</net>
-<net name="LED_B" class="0">
-<segment>
-<pinref part="U$1" gate="G$1" pin="35"/>
-<wire x1="66.04" y1="58.42" x2="81.28" y2="58.42" width="0.1524" layer="91"/>
-<label x="68.58" y="58.42" size="1.778" layer="95"/>
-</segment>
-<segment>
-<pinref part="R2" gate="G$1" pin="1"/>
-<wire x1="116.84" y1="81.28" x2="109.22" y2="81.28" width="0.1524" layer="91"/>
-<label x="109.22" y="81.28" size="1.778" layer="95"/>
 </segment>
 </net>
@@
 <segment>
 <pinref part="C1" gate="G$1" pin="-"/>
+<pinref part="RCA_HOT" gate="A" pin="2"/>
 <wire x1="172.72" y1="55.88" x2="177.8" y2="55.88" width="0.1524" layer="91"/>
-<pinref part="RCA_HOT" gate="A" pin="1"/>
-</segment>
-</net>
+</segment>
+</net>
+<net name="I2C_SDA" class="0">
+<segment>
+<pinref part="U$1" gate="G$1" pin="50"/>
+<wire x1="66.04" y1="96.52" x2="81.28" y2="96.52" width="0.1524" layer="91"/>
+<label x="68.58" y="96.52" size="1.778" layer="95"/>
+</segment>
+<segment>
+<pinref part="JP1" gate="A" pin="5"/>
+<wire x1="220.98" y1="124.46" x2="205.74" y2="124.46" width="0.1524" layer="91"/>
+<label x="205.74" y="124.46" size="1.778" layer="95"/>
+</segment>
+</net>
+<net name="I2C_SCL" class="0">
+<segment>
+<pinref part="U$1" gate="G$1" pin="49"/>
+<wire x1="66.04" y1="93.98" x2="81.28" y2="93.98" width="0.1524" layer="91"/>
+<label x="68.58" y="93.98" size="1.778" layer="95"/>
+</segment>
+<segment>
+<pinref part="JP1" gate="A" pin="4"/>
+<wire x1="220.98" y1="127" x2="205.74" y2="127" width="0.1524" layer="91"/>
+<label x="205.74" y="127" size="1.778" layer="95"/>
+</segment>
+</net>

Commit message: Eagle: 修正
Parts:
- R1, R2: value (none) -> 1k
- R3: value (none) -> 1.5k
- R4, R6: value (none) -> 220
- R5: value (none) -> 10k
Connections:
- net VDAC8_1: now also U$1.22; no longer R6.2, U$1.23
- net VDAC8_2: now also R6.2, U$1.23; no longer U$1.24
Other:
- moved on the sheet: LED1, R6, TP4
Changed lines of the file:
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@@
 <?xml version="1.0" encoding="utf-8"?>
 <!DOCTYPE eagle SYSTEM "eagle.dtd">
-<eagle version="7.5.0">
+<eagle version="7.2.0">
 <drawing>
 <settings>
@@
 <setting verticaltext="up"/>
 </settings>
-<grid distance="0.1" unitdist="inch" unit="inch" style="dots" multiple="1" display="yes" altdistance="0.01" altunitdist="inch" altunit="inch"/>
+<grid distance="0.1" unitdist="inch" unit="inch" style="lines" multiple="1" display="no" altdistance="0.01" altunitdist="inch" altunit="inch"/>
 <layers>
 <layer number="1" name="Top" color="4" fill="1" visible="no" active="no"/>
@@
 <part name="SUPPLY10" library="supply2" deviceset="GND" device=""/>
 <part name="RGB_LED" library="pinhead" deviceset="PINHD-1X4" device=""/>
-<part name="R1" library="rcl" deviceset="R-EU_" device="0207/7"/>
-<part name="R2" library="rcl" deviceset="R-EU_" device="0207/7"/>
-<part name="R3" library="rcl" deviceset="R-EU_" device="0207/7"/>
+<part name="R1" library="rcl" deviceset="R-EU_" device="0207/7" value="1k"/>
+<part name="R2" library="rcl" deviceset="R-EU_" device="0207/7" value="1k"/>
+<part name="R3" library="rcl" deviceset="R-EU_" device="0207/7" value="1.5k"/>
 <part name="SUPPLY13" library="supply2" deviceset="GND" device=""/>
 <part name="JP1" library="pinhead" deviceset="PINHD-1X5" device="/90" value="SEQUENCER"/>
@@
 <part name="JP3" library="pinhead" deviceset="PINHD-1X5" device="/90" value="SPI"/>
 <part name="SUPPLY18" library="supply2" deviceset="GND" device=""/>
-<part name="R4" library="rcl" deviceset="R-EU_" device="0207/7"/>
+<part name="R4" library="rcl" deviceset="R-EU_" device="0207/7" value="220"/>
 <part name="VCC5" library="supply1" deviceset="VCCIO" device=""/>
-<part name="R5" library="rcl" deviceset="R-TRIMM" device="3339P"/>
+<part name="R5" library="rcl" deviceset="R-TRIMM" device="3339P" value="10k"/>
 <part name="SUPPLY19" library="supply2" deviceset="GND" device=""/>
 <part name="SUPPLY20" library="supply2" deviceset="GND" device=""/>
-<part name="R6" library="rcl" deviceset="R-EU_" device="0207/7"/>
+<part name="R6" library="rcl" deviceset="R-EU_" device="0207/7" value="220"/>
 <part name="LED1" library="led" deviceset="LED" device="3MM"/>
 <part name="SUPPLY21" library="supply2" deviceset="GND" device=""/>
@@
 <instance part="SUPPLY19" gate="GND" x="30.48" y="109.22"/>
 <instance part="SUPPLY20" gate="GND" x="190.5" y="33.02"/>
-<instance part="R6" gate="G$1" x="160.02" y="48.26" rot="R90"/>
-<instance part="LED1" gate="G$1" x="160.02" y="40.64"/>
-<instance part="SUPPLY21" gate="GND" x="160.02" y="33.02"/>
+<instance part="R6" gate="G$1" x="144.78" y="48.26" rot="R90"/>
+<instance part="LED1" gate="G$1" x="144.78" y="40.64"/>
+<instance part="SUPPLY21" gate="GND" x="144.78" y="33.02"/>
 <instance part="C1" gate="G$1" x="167.64" y="55.88" rot="R90"/>
 <instance part="RCA_HOT" gate="A" x="180.34" y="50.8"/>
@@
 <instance part="TP2" gate="G$1" x="93.98" y="93.98" rot="R180"/>
 <instance part="TP3" gate="G$1" x="25.4" y="50.8"/>
-<instance part="TP4" gate="G$1" x="35.56" y="50.8"/>
+<instance part="TP4" gate="G$1" x="132.08" y="60.96"/>
 </instances>
 <busses>
@@
 <net name="VDAC8_2" class="0">
 <segment>
-<pinref part="U$1" gate="G$1" pin="24"/>
-<wire x1="50.8" y1="43.18" x2="35.56" y2="43.18" width="0.1524" layer="91"/>
-<label x="38.1" y="43.18" size="1.778" layer="95"/>
 <pinref part="TP4" gate="G$1" pin="TP"/>
-<wire x1="35.56" y1="48.26" x2="35.56" y2="43.18" width="0.1524" layer="91"/>
-</segment>
-</net>
-<net name="VDAC8_1" class="0">
+<wire x1="132.08" y1="58.42" x2="132.08" y2="55.88" width="0.1524" layer="91"/>
+</segment>
 <segment>
 <pinref part="U$1" gate="G$1" pin="23"/>
@@
 <segment>
 <pinref part="R6" gate="G$1" pin="2"/>
-<wire x1="160.02" y1="53.34" x2="160.02" y2="55.88" width="0.1524" layer="91"/>
+<wire x1="144.78" y1="53.34" x2="144.78" y2="55.88" width="0.1524" layer="91"/>
+<wire x1="144.78" y1="55.88" x2="132.08" y2="55.88" width="0.1524" layer="91"/>
+<label x="132.08" y="55.88" size="1.778" layer="95"/>
+</segment>
+</net>
+<net name="VDAC8_1" class="0">
+<segment>
 <pinref part="C1" gate="G$1" pin="+"/>
-<wire x1="160.02" y1="55.88" x2="165.1" y2="55.88" width="0.1524" layer="91"/>
-<label x="160.02" y="58.42" size="1.778" layer="95" rot="R180"/>
-</segment>
-</net>
+<wire x1="149.86" y1="55.88" x2="165.1" y2="55.88" width="0.1524" layer="91"/>
+<label x="162.56" y="58.42" size="1.778" layer="95" rot="R180"/>
+</segment>
+<segment>
+<pinref part="U$1" gate="G$1" pin="22"/>
+<wire x1="50.8" y1="48.26" x2="38.1" y2="48.26" width="0.1524" layer="91"/>
+<label x="38.1" y="48.26" size="1.778" layer="95"/>
+</segment>
+</net>

Commit message: Eagleファイル修正
Connections:
- removed net SW3: U$1.4
- removed net SW4: U$1.5
Changed lines of the file:
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@@
-</segment>
-</net>
-<net name="SW3" class="0">
-<segment>
-<pinref part="U$1" gate="G$1" pin="4"/>
-<wire x1="38.1" y1="93.98" x2="50.8" y2="93.98" width="0.1524" layer="91"/>
-<label x="38.1" y="93.98" size="1.778" layer="95"/>
-</segment>
-</net>
-<net name="SW4" class="0">
-<segment>
-<pinref part="U$1" gate="G$1" pin="5"/>
-<wire x1="38.1" y1="91.44" x2="50.8" y2="91.44" width="0.1524" layer="91"/>
-<label x="38.1" y="91.44" size="1.778" layer="95"/>
 </segment>
 </net>
